File: hardware/MeteoNet.kicad_sch (KiCad schematic)
At the start: 6 parts, among them Q1 XC6220B331MR-G, U1 ESP32-S3-WROOM-1

Commit message: PCB
Parts:
- added C1: 1uF, Capacitor_SMD:C_0603_1608Metric, symbol JLCPCB_Capacitors:CL10A106KP8NNNC
- added C4: 100nF, Capacitor_SMD:C_0603_1608Metric, symbol JLCPCB_Capacitors:CL05B104KO5NNNC
- added C6: 1uF, Capacitor_SMD:C_0603_1608Metric, symbol JLCPCB_Capacitors:CL05B104KO5NNNC
- added C8: 10uF, Capacitor_SMD:C_0805_2012Metric, symbol JLCPCB_Capacitors:CL05B104KO5NNNC
- added C9: 4,7uF, Capacitor_SMD:C_0805_2012Metric, symbol JLCPCB_Capacitors:CL05B104KO5NNNC
- added FID1, FID2, FID3: Fiducial, Fiducial:Fiducial_1mm_Mask2mm, symbol Mechanical:Fiducial
- added H1, H2, H3, H4: MountingHole, MountingHole:MountingHole_2.5mm_Pad, symbol Mechanical:MountingHole
- added J1: USB_C_Receptacle_USB2.0_16P, Connector_USB:USB_C_Receptacle_HRO_TYPE-C-31-M-12, symbol Connector:USB_C_Receptacle_USB2.0_16P
- added J2: BAT, Connector_JST:JST_PH_B2B-PH-SM4-TB_1x02-1MP_P2.00mm_Vertical, symbol Connector_Generic:Conn_01x02
- added J3: DS18B20, Connector_PinSocket_2.54mm:PinSocket_1x03_P2.54mm_Vertical_SMD_Pin1Left, symbol Connector_Generic:Conn_01x03
- added J4: BME280, Connector_PinSocket_2.54mm:PinSocket_1x04_P2.54mm_Vertical_SMD_Pin1Left, symbol Connector_Generic:Conn_01x04
- added Q1: BSS138, Package_TO_SOT_SMD:SOT-23, symbol Transistor_FET:BSS138
- added Q2: BSS84, Package_TO_SOT_SMD:SOT-23, symbol Transistor_FET:BSS84
- added R1, R11, R2, R7: 10k, Resistor_SMD:R_0603_1608Metric, symbol Device:R
- added R10, R8, R9: 100k, Resistor_SMD:R_0603_1608Metric, symbol Device:R
- added R12: 4k7, Resistor_SMD:R_0603_1608Metric, symbol Device:R
- added R3, R4: 5k1, Resistor_SMD:R_0603_1608Metric, symbol Device:R
- added R5: 1k2, Resistor_SMD:R_0603_1608Metric, symbol Device:R
- added R6: 1k5, Resistor_SMD:R_0603_1608Metric, symbol Device:R
- added SW1: BTN_EN, Button_Switch_SMD:SW_SPST_PTS645Sx43SMTR92, symbol Switch:SW_Push
- added SW2: BTN_IO0, Button_Switch_SMD:SW_SPST_PTS645Sx43SMTR92, symbol Switch:SW_Push
- added TP1: TXD0, TestPoint:TestPoint_Pad_D1.5mm, symbol Connector:TestPoint
- added TP2: RXD0, TestPoint:TestPoint_Pad_D1.5mm, symbol Connector:TestPoint
- added TP3: GND, TestPoint:TestPoint_Pad_D1.5mm, symbol Connector:TestPoint
- added TP4: LDO_3V3, TestPoint:TestPoint_Pad_D1.5mm, symbol Connector:TestPoint
- added TP5: VBAT, TestPoint:TestPoint_Pad_D1.5mm, symbol Connector:TestPoint
- added TP6: USB_VBUS, TestPoint:TestPoint_Pad_D1.5mm, symbol Connector:TestPoint
- added U2: USBLC6-2SC6, Package_TO_SOT_SMD:SOT-23-6, symbol Power_Protection:USBLC6-2SC6
- added U3: BQ24072RGT, Package_DFN_QFN:VQFN-16-1EP_3x3mm_P0.5mm_EP1.6x1.6mm, symbol Battery_Management:BQ24072RGT
- C2: renamed from C3; footprint PCM_JLCPCB_Capacitors:C0603 -> Capacitor_SMD:C_0805_2012Metric; LCSC Part # (none) -> C15850
- C3: renamed from C4; footprint PCM_JLCPCB_Capacitors:C0402 -> Capacitor_SMD:C_0603_1608Metric; LCSC Part # (none) -> C14663
- C5: renamed from C1; footprint PCM_JLCPCB_Capacitors:C0603 -> Capacitor_SMD:C_0805_2012Metric; LCSC Part # (none) -> C15850
- C7: renamed from C2; footprint PCM_JLCPCB_Capacitors:C0603 -> Capacitor_SMD:C_0805_2012Metric; LCSC Part # (none) -> C15850
- Q3: renamed from Q1; footprint PCM_JLCPCB_Power_Management_ICs:SOT-25_L3.0-W1.6-P0.95-LS2.8-TL -> Package_TO_SOT_SMD:SOT-23-5; LCSC Part # (none) -> C86534
- U1: LCSC Part # (none) -> C2913198
Connections:
- net GND: now also C1.1, C4.2, C6.1, C8.1, C9.1, J1.A1 (GND), J1.A12 (GND), J1.B1 (GND), J1.B12 (GND), J1.SH (SHIELD), J2.2 (Pin_2), J3.1 (Pin_1), J4.2 (Pin_2), Q1.2 (S), R11.1, R3.1, R4.2, R5.2, R6.2, SW1.2, SW2.2, TP3.1, U2.2 (GND), U3.14 (TMR), U3.15 (TD), U3.17 (VSS), U3.4 (~{CE}), U3.6 (EN1), U3.8 (VSS)
- net LDO_3V3: now also Q2.2 (S), R1.2, R2.1, R8.1, TP4.1
- net LDO_VIN: now also C8.2, U3.10 (OUT), U3.11 (OUT), U3.5 (EN2)
- net USB_D-: now reaches U1.13 (USB_D-)
- net USB_D-: now also U2.6 (I/O1)
- net USB_D+: now reaches U1.14 (USB_D+)
- net USB_D+: now also U2.4 (I/O2)
- net IO9: now reaches U1.17 (IO9)
- net IO9: now also J3.2 (Pin_2), R12.2
- net IO10: now reaches U1.18 (IO10)
- net IO10: now also J4.3 (Pin_3)
- net IO11: now reaches U1.19 (IO11)
- net IO11: now also J4.4 (Pin_4)
- net IO12: now reaches U1.20 (IO12)
- net IO12: now also R7.2
- net IO0: now reaches U1.27 (IO0)
- net IO0: now also R2.2, SW2.1
- net EN: now reaches U1.3 (EN)
- net EN: now also C1.2, R1.1, SW1.1
- net RXD0: now reaches U1.36 (RXD0)
- net RXD0: now also TP2.1
- net TXD0: now reaches U1.37 (TXD0)
- net TXD0: now also TP1.1
- net IO4: now reaches U1.4 (IO4)
- net IO4: now also U3.9 (~{CHG})
- net IO5: now reaches U1.5 (IO5)
- net IO5: now also U3.7 (~{PGOOD})
- net IO6: now reaches U1.6 (IO6)
- net IO6: now also R10.2, R9.1
- net IO7: now reaches U1.7 (IO7)
- net IO7: now also Q1.1 (G)
- new net: J1.A5 (CC1), R3.2
- new net: J1.B5 (CC2), R4.1
- new net: Q2.1 (G), R7.1, R8.2
- new net: Q1.3 (D), R10.1
- new net: R11.2, U3.1 (TS)
- new net: R5.1, U3.12 (ILIM)
- new net: R6.1, U3.16 (ISET)
- new net: J1.A7 (D-), J1.B7 (D-), U2.1 (I/O1)
- new net: J1.A6 (D+), J1.B6 (D+), U2.3 (I/O2)
- new net USB_VBUS: C4.1, C6.2, J1.A4 (VBUS), J1.A9 (VBUS), J1.B4 (VBUS), J1.B9 (VBUS), TP6.1, U2.5 (VBUS), U3.13 (IN)
- new net VBAT: C9.2, J2.1 (Pin_1), R9.2, TP5.1, U3.2 (BAT), U3.3 (BAT)
- new net VCC_SENS: J3.3 (Pin_3), J4.1 (Pin_1), Q2.3 (D), R12.1
- no-connect marks 1 -> 26
Other:
- moved on the sheet: C2, C3, C5, C7, Q3, U1

Commit message: PCB routing
Connections:
- net GND: now also C9.2; no longer C9.1
- net IO6: now also Q1.1 (G); no longer R10.2, R9.1
- net IO7: now also R10.2, R9.1; no longer Q1.1 (G)
- net VBAT: now also C9.1; no longer C9.2
Changed lines of the file:
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@@
 	)
 	(label "IO6"
-		(at 160.02 158.75 180)
+		(at 160.02 175.26 180)
 		(effects
 			(font
@@
 	)
 	(label "IO7"
-		(at 160.02 175.26 180)
+		(at 160.02 158.75 180)
 		(effects
 			(font
@@
 		(lib_id "JLCPCB_Capacitors:CL05B104KO5NNNC")
 		(at 201.93 224.79 0)
-		(mirror y)
 		(unit 1)
 		(body_style 1)
