File: hardware/MeteoNet.kicad_pcb (KiCad board)
At the start: 2 copper layers, 0 parts

Commit message: PCB
Parts:
- added C1: 1uF, Capacitor_SMD:C_0603_1608Metric, F.Cu at (145.1, 65.5)
- added C2: 10uF, Capacitor_SMD:C_0805_2012Metric, F.Cu at (145.1, 70.1)
- added C3: 100nF, Capacitor_SMD:C_0603_1608Metric, F.Cu at (145.6, 72.7)
- added C4: 100nF, Capacitor_SMD:C_0603_1608Metric, F.Cu at (102.6, 77.6)
- added C5: 10uF, Capacitor_SMD:C_0805_2012Metric, F.Cu at (118.0, 66.1)
- added C6: 1uF, Capacitor_SMD:C_0603_1608Metric, F.Cu at (110.5, 65.2)
- added C7: 10uF, Capacitor_SMD:C_0805_2012Metric, F.Cu at (126.8, 66.1)
- added C8: 10uF, Capacitor_SMD:C_0805_2012Metric, F.Cu at (113.7, 64.2)
- added C9: 4,7uF, Capacitor_SMD:C_0805_2012Metric, F.Cu at (114.6, 72.0)
- added FID1: Fiducial, Fiducial:Fiducial_1mm_Mask2mm, F.Cu at (99.6, 63.5)
- added FID2: Fiducial, Fiducial:Fiducial_1mm_Mask2mm, F.Cu at (147.6, 63.5)
- added FID3: Fiducial, Fiducial:Fiducial_1mm_Mask2mm, F.Cu at (99.5, 100.0)
- added H1: MountingHole, MountingHole:MountingHole_2.5mm_Pad, F.Cu at (95.0, 65.0)
- added H2: MountingHole, MountingHole:MountingHole_2.5mm_Pad, F.Cu at (152.2, 65.0)
- added H3: MountingHole, MountingHole:MountingHole_2.5mm_Pad, F.Cu at (95.0, 98.5)
- added H4: MountingHole, MountingHole:MountingHole_2.5mm_Pad, F.Cu at (152.2, 98.5)
- added J1: USB_C_Receptacle_USB2.0_16P, Connector_USB:USB_C_Receptacle_HRO_TYPE-C-31-M-12, F.Cu at (94.0, 74.3)
- added J2: BAT, Connector_JST:JST_PH_B2B-PH-SM4-TB_1x02-1MP_P2.00mm_Vertical, F.Cu at (94.7, 86.7)
- added J3: DS18B20, Connector_PinSocket_2.54mm:PinSocket_1x03_P2.54mm_Vertical_SMD_Pin1Left, F.Cu at (112.5, 99.7)
- added J4: BME280, Connector_PinSocket_2.54mm:PinSocket_1x04_P2.54mm_Vertical_SMD_Pin1Left, F.Cu at (124.3, 99.7)
- added Q1: BSS138, Package_TO_SOT_SMD:SOT-23, F.Cu at (104.1, 92.7)
- added Q2: BSS84, Package_TO_SOT_SMD:SOT-23, F.Cu at (115.3, 78.9)
- added Q3: XC6220B331MR-G, Package_TO_SOT_SMD:SOT-23-5, F.Cu at (122.4, 66.1)
- added R1: 10k, Resistor_SMD:R_0603_1608Metric, F.Cu at (141.7, 72.7)
- added R10: 100k, Resistor_SMD:R_0603_1608Metric, F.Cu at (101.0, 92.8)
- added R11: 10k, Resistor_SMD:R_0603_1608Metric, F.Cu at (108.4, 71.9)
- added R12: 4k7, Resistor_SMD:R_0603_1608Metric, F.Cu at (111.7, 95.6)
- added R2: 10k, Resistor_SMD:R_0603_1608Metric, F.Cu at (125.5, 93.5)
- added R3: 5k1, Resistor_SMD:R_0603_1608Metric, F.Cu at (100.9, 68.2)
- added R4: 5k1, Resistor_SMD:R_0603_1608Metric, F.Cu at (100.9, 80.4)
- added R5: 1k2, Resistor_SMD:R_0603_1608Metric, F.Cu at (109.8, 62.9)
- added R6: 1k5, Resistor_SMD:R_0603_1608Metric, F.Cu at (108.4, 70.3)
- added R7: 10k, Resistor_SMD:R_0603_1608Metric, F.Cu at (119.3, 81.2)
- added R8: 100k, Resistor_SMD:R_0603_1608Metric, F.Cu at (119.3, 78.4)
- added R9: 100k, Resistor_SMD:R_0603_1608Metric, F.Cu at (101.0, 89.7)
- added SW1: BTN_EN, Button_Switch_SMD:SW_SPST_PTS645Sx43SMTR92, F.Cu at (138.7, 64.0)
- added SW2: BTN_IO0, Button_Switch_SMD:SW_SPST_PTS645Sx43SMTR92, F.Cu at (138.7, 99.4)
- added TP1: TXD0, TestPoint:TestPoint_Pad_D1.5mm, F.Cu at (41.5, 61.2)
- added TP2: RXD0, TestPoint:TestPoint_Pad_D1.5mm, F.Cu at (41.5, 64.8)
- added TP3: GND, TestPoint:TestPoint_Pad_D1.5mm, F.Cu at (41.5, 68.3)
- added TP4: LDO_3V3, TestPoint:TestPoint_Pad_D1.5mm, F.Cu at (45.1, 61.2)
- added TP5: VBAT, TestPoint:TestPoint_Pad_D1.5mm, F.Cu at (45.1, 64.8)
- added TP6: USB_VBUS, TestPoint:TestPoint_Pad_D1.5mm, F.Cu at (45.1, 68.3)
- added U1: ESP32-S3-WROOM-1, RF_Module:ESP32-S3-WROOM-1, F.Cu at (140.9, 84.5)
- added U2: USBLC6-2SC6, Package_TO_SOT_SMD:SOT-23-6, F.Cu at (102.6, 74.3)
- added U3: BQ24072RGT, Package_DFN_QFN:VQFN-16-1EP_3x3mm_P0.5mm_EP1.6x1.6mm, F.Cu at (113.4, 68.3)
Routing:
- net /LDO_3V3: track 0.00 -> 69.4 mm, vias 0 -> 2
- net /VCC_SENS: track 0.00 -> 38.3 mm
- net /USB_VBUS: track 0.00 -> 33.1 mm
- net /IO4: track 0.00 -> 32.7 mm, vias 0 -> 2
- net /VBAT: track 0.00 -> 31.6 mm, vias 0 -> 2
- net /IO5: track 0.00 -> 30.1 mm, vias 0 -> 2
- net /USB_D-: track 0.00 -> 28.3 mm
- net /USB_D+: track 0.00 -> 28.1 mm
- net /EN: track 0.00 -> 23.2 mm, vias 0 -> 2
- net /LDO_VIN: track 0.00 -> 19.0 mm
- net /IO0: track 0.00 -> 18.3 mm
- net GND: track 0.00 -> 10.9 mm, vias 0 -> 5
- net Net-(J1-CC1): track 0.00 -> 6.79 mm, vias 0 -> 2
- net Net-(J1-CC2): track 0.00 -> 6.40 mm, vias 0 -> 2
- net Net-(Q2-G): track 0.00 -> 6.31 mm
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- added copper zone on B.Cu, net GND
- added copper zone on F.Cu, net GND
Other:
- board outline added: 67.3 x 43.5 mm

Commit message: PCB routing
Parts:
- moved Q1 0.94 mm to (104.1, 93.7), turned to 180 degrees
- turned C9 to 0 degrees
Connections:
- C9 pad 1: GND -> /VBAT
- C9 pad 2: /VBAT -> GND
- Q1 pad 1: /IO7 -> /IO6
- R10 pad 2: /IO6 -> /IO7
- R9 pad 1: /IO6 -> /IO7
Routing:
- net /IO7: track 0.00 -> 47.2 mm, vias 0 -> 4
- net /IO6: track 1.45 -> 44.0 mm, vias 0 -> 4
- net /IO9: track 5.90 -> 35.9 mm, vias 0 -> 2
- net /IO11: track 0.00 -> 24.5 mm, vias 0 -> 2
- net /IO10: track 0.00 -> 20.8 mm, vias 0 -> 2
- net /IO12: track 0.00 -> 9.42 mm, vias 0 -> 2
- net GND: track 10.9 -> 14.2 mm, vias 5 -> 29
- net Net-(Q1-D): track 3.07 -> 2.13 mm
- net /VCC_SENS: track 38.3 -> 38.8 mm

Commit message: TP value -> F.silkscreen
Parts:
- moved TP4 5.25 mm to (46.6, 56.2)
- moved TP1 5.00 mm to (41.5, 56.2)
- moved TP5 3.82 mm to (47.0, 61.5)
- moved TP2 3.30 mm to (41.5, 61.5)
- moved TP6 2.83 mm to (47.4, 66.7)
- moved TP3 1.70 mm to (41.5, 66.6)
Changed lines of the file:
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@@
 	(footprint "TestPoint:TestPoint_Pad_D1.5mm"
 		(layer "F.Cu")
-		(at 41.505 68.325)
+		(at 41.505 66.625)
 		(descr "SMD pad as test Point, diameter 1.5mm")
 		(tags "test point SMD pad")
@@
 		(property "Value" "GND"
 			(at 0 1.75 0)
-			(layer "F.Fab")
+			(layer "F.SilkS")
 			(effects
 				(font
@@
 		(tags "Surface mounted socket strip SMD 1x04 2.54mm single row style1 pin1 left")
 		(property "Reference" "J4"
-			(at 0 -6.68 90)
+			(at -0.015 -6.44 90)
 			(layer "F.SilkS")
 			(effects
@@
 		)
 		(property "Value" "BME280"
-			(at 0 6.68 90)
-			(layer "F.Fab")
+			(at 0 6.285 90)
+			(layer "F.SilkS")
 			(effects
 				(font
@@
 	(footprint "TestPoint:TestPoint_Pad_D1.5mm"
 		(layer "F.Cu")
-		(at 41.505 64.775)
+		(at 41.505 61.475)
 		(descr "SMD pad as test Point, diameter 1.5mm")
 		(tags "test point SMD pad")
@@
 		(property "Value" "RXD0"
 			(at 0 1.75 0)
-			(layer "F.Fab")
+			(layer "F.SilkS")
 			(effects
 				(font
@@
 		(tags "Surface mounted socket strip SMD 1x03 2.54mm single row style1 pin1 left")
 		(property "Reference" "J3"
-			(at 0 -5.41 90)
+			(at -0.0125 6.315 90)
 			(layer "F.SilkS")
 			(effects
@@
 		)
 		(property "Value" "DS18B20"
-			(at 0 5.41 90)
-			(layer "F.Fab")
+			(at -0.0125 5.065 90)
+			(layer "F.SilkS")
 			(effects
 				(font
@@
 	(footprint "TestPoint:TestPoint_Pad_D1.5mm"
 		(layer "F.Cu")
-		(at 41.505 61.225)
+		(at 41.505 56.225)
 		(descr "SMD pad as test Point, diameter 1.5mm")
 		(tags "test point SMD pad")
@@
 		(property "Value" "TXD0"
 			(at 0 1.75 0)
-			(layer "F.Fab")
+			(layer "F.SilkS")
 			(effects
 				(font
@@
 	(footprint "TestPoint:TestPoint_Pad_D1.5mm"
 		(layer "F.Cu")
-		(at 45.055 68.325)
+		(at 47.35 66.675)
 		(descr "SMD pad as test Point, diameter 1.5mm")
 		(tags "test point SMD pad")
@@
 		(property "Value" "USB_VBUS"
 			(at 0 1.75 0)
-			(layer "F.Fab")
+			(layer "F.SilkS")
 			(effects
 				(font
@@
 	(footprint "TestPoint:TestPoint_Pad_D1.5mm"
 		(layer "F.Cu")
-		(at 45.055 61.225)
+		(at 46.65 56.225)
 		(descr "SMD pad as test Point, diameter 1.5mm")
 		(tags "test point SMD pad")
@@
 		(property "Value" "LDO_3V3"
 			(at 0 1.75 0)
-			(layer "F.Fab")
+			(layer "F.SilkS")
 			(effects
 				(font
@@
 	(footprint "TestPoint:TestPoint_Pad_D1.5mm"
 		(layer "F.Cu")
-		(at 45.055 64.775)
+		(at 47.025 61.5)
 		(descr "SMD pad as test Point, diameter 1.5mm")
 		(tags "test point SMD pad")
@@
 		(property "Value" "VBAT"
 			(at 0 1.75 0)
-			(layer "F.Fab")
+			(layer "F.SilkS")
 			(effects
 				(font
